File: pcb/leds.kicad_sch (KiCad schematic)
At the start: 29 parts, among them U10 LDS-C814RI, U11 LDS-C814RI, U12 74HC595, U13 74HC595, U14 74HC595, U15 LDS-C814RI, U16 LDS-R8006RI, U6 74HC595, U7 74HC595, U8 74HC595, U9 LDS-C814RI

Commit message: Laid out and routed PCB
Parts:
- RN1, RN10, RN11, RN12, RN2, RN3, RN4, RN5, RN6, RN7, RN8, RN9: footprint (none) -> Resistor_SMD:R_Array_Convex_4x0603
- U12, U13, U14, U6, U7, U8: footprint (none) -> Package_SO:SOIC-16_3.9x9.9mm_P1.27mm
Connections:
- net at RN12.1 (R1.1): now also U16.3 (K); no longer U16.5 (U)
- net at RN12.2 (R2.1): now also U16.2 (M); no longer U16.7 (T)
- net at RN12.3 (R3.1): now also U16.17 (N); no longer U16.14 (R)
- net at RN12.4 (R4.1): now also U16.15 (P); no longer U16.6 (S)
- net at RN12.5 (R4.2): now also U14.3 (QD); no longer U14.4 (QE)
- net at RN12.6 (R3.2): now also U14.2 (QC); no longer U14.5 (QF)
- net at RN12.7 (R2.2): now also U14.1 (QB); no longer U14.6 (QG)
- net at RN12.8 (R1.2): now also U14.15 (QA); no longer U14.7 (QH)
- net at U10.1 (A): now also RN4.1 (R1.1); no longer RN3.4 (R4.1)
- net at U10.10 (D): now also RN4.4 (R4.1); no longer RN3.1 (R1.1)
- net at U10.12 (C): now also RN4.3 (R3.1); no longer RN3.2 (R2.1)
- net at U10.13 (G): now also RN3.3 (R3.1); no longer RN4.2 (R2.1)
- net at U10.14 (B): now also RN4.2 (R2.1); no longer RN3.3 (R3.1)
- net at U10.2 (F): now also RN3.2 (R2.1); no longer RN4.3 (R3.1)
- net at U10.4 (E): now also RN3.1 (R1.1); no longer RN4.4 (R4.1)
- net at U10.6 (LDP): now also RN3.4 (R4.1); no longer RN4.1 (R1.1)
- net at RN11.1 (R1.1): now also U16.6 (S); no longer U16.15 (P)
- net at RN11.2 (R2.1): now also U16.14 (R); no longer U16.17 (N)
- net at RN11.3 (R3.1): now also U16.7 (T); no longer U16.2 (M)
- net at RN11.4 (R4.1): now also U16.5 (U); no longer U16.3 (K)
- net at RN11.5 (R4.2): now also U14.7 (QH); no longer U14.15 (QA)
- net at RN11.6 (R3.2): now also U14.6 (QG); no longer U14.1 (QB)
- net at RN11.7 (R2.2): now also U14.5 (QF); no longer U14.2 (QC)
- net at RN11.8 (R1.2): now also U14.4 (QE); no longer U14.3 (QD)
- net at RN2.1 (R1.1): now also U9.1 (A); no longer U9.6 (LDP)
- net at RN2.2 (R2.1): now also U9.14 (B); no longer U9.13 (G)
- net at RN2.3 (R3.1): now also U9.12 (C); no longer U9.2 (F)
- net at RN2.4 (R4.1): now also U9.10 (D); no longer U9.4 (E)
- net at RN2.5 (R4.2): now also U6.3 (QD); no longer U6.4 (QE)
- net at RN2.6 (R3.2): now also U6.2 (QC); no longer U6.5 (QF)
- net at RN2.7 (R2.2): now also U6.1 (QB); no longer U6.6 (QG)
- net at RN2.8 (R1.2): now also U6.15 (QA); no longer U6.7 (QH)
- net at RN1.6 (R3.2): now also U6.6 (QG); no longer U6.1 (QB)
- net at RN1.5 (R4.2): now also U6.7 (QH); no longer U6.15 (QA)
- net at RN1.7 (R2.2): now also U6.5 (QF); no longer U6.2 (QC)
- net at RN1.8 (R1.2): now also U6.4 (QE); no longer U6.3 (QD)
- net at RN1.4 (R4.1): now also U9.6 (LDP); no longer U9.1 (A)
- net at RN1.1 (R1.1): now also U9.4 (E); no longer U9.10 (D)
- net at RN1.2 (R2.1): now also U9.2 (F); no longer U9.12 (C)
- net at RN1.3 (R3.1): now also U9.13 (G); no longer U9.14 (B)
- net at U12.1 (QB): now also RN8.7 (R2.2); no longer RN7.6 (R3.2)
- net at U12.15 (QA): now also RN8.8 (R1.2); no longer RN7.5 (R4.2)
- net at U12.2 (QC): now also RN8.6 (R3.2); no longer RN7.7 (R2.2)
- net at U12.3 (QD): now also RN8.5 (R4.2); no longer RN7.8 (R1.2)
- net at U12.4 (QE): now also RN7.8 (R1.2); no longer RN8.5 (R4.2)
- net at U12.5 (QF): now also RN7.7 (R2.2); no longer RN8.6 (R3.2)
- net at U12.6 (QG): now also RN7.6 (R3.2); no longer RN8.7 (R2.2)
- net at U12.7 (QH): now also RN7.5 (R4.2); no longer RN8.8 (R1.2)
- net at U15.1 (A): now also RN8.1 (R1.1); no longer RN7.4 (R4.1)
- net at U15.10 (D): now also RN8.4 (R4.1); no longer RN7.1 (R1.1)
- net at U15.12 (C): now also RN8.3 (R3.1); no longer RN7.2 (R2.1)
- net at U15.13 (G): now also RN7.3 (R3.1); no longer RN8.2 (R2.1)
- net at U15.14 (B): now also RN8.2 (R2.1); no longer RN7.3 (R3.1)
- net at U15.2 (F): now also RN7.2 (R2.1); no longer RN8.3 (R3.1)
- net at U15.4 (E): now also RN7.1 (R1.1); no longer RN8.4 (R4.1)
- net at U15.6 (LDP): now also RN7.4 (R4.1); no longer RN8.1 (R1.1)
- net at U13.1 (QB): now also RN10.7 (R2.2); no longer RN9.6 (R3.2)
- net at U13.15 (QA): now also RN10.8 (R1.2); no longer RN9.5 (R4.2)
- net at U13.2 (QC): now also RN10.6 (R3.2); no longer RN9.7 (R2.2)
- net at U13.3 (QD): now also RN10.5 (R4.2); no longer RN9.8 (R1.2)
- net at U13.4 (QE): now also RN9.8 (R1.2); no longer RN10.5 (R4.2)
- net at U13.5 (QF): now also RN9.7 (R2.2); no longer RN10.6 (R3.2)
- net at U13.6 (QG): now also RN9.6 (R3.2); no longer RN10.7 (R2.2)
- net at U13.7 (QH): now also RN9.5 (R4.2); no longer RN10.8 (R1.2)
- net at RN9.1 (R1.1): now also U16.10 (E); no longer U16.13 (D)
- net at RN9.2 (R2.1): now also U16.9 (F); no longer U16.16 (C)
- net at RN9.3 (R3.1): now also U16.8 (G); no longer U16.18 (B)
- net at RN9.4 (R4.1): now also U16.4 (H); no longer U16.1 (A)
- net at U8.1 (QB): now also RN6.7 (R2.2); no longer RN5.6 (R3.2)
- net at U8.15 (QA): now also RN6.8 (R1.2); no longer RN5.5 (R4.2)
- net at U8.2 (QC): now also RN6.6 (R3.2); no longer RN5.7 (R2.2)
- net at U8.3 (QD): now also RN6.5 (R4.2); no longer RN5.8 (R1.2)
- net at U8.4 (QE): now also RN5.8 (R1.2); no longer RN6.5 (R4.2)
- net at U8.5 (QF): now also RN5.7 (R2.2); no longer RN6.6 (R3.2)
- net at U8.6 (QG): now also RN5.6 (R3.2); no longer RN6.7 (R2.2)
- net at U8.7 (QH): now also RN5.5 (R4.2); no longer RN6.8 (R1.2)
- net at U7.1 (QB): now also RN4.7 (R2.2); no longer RN3.6 (R3.2)
- net at U7.15 (QA): now also RN4.8 (R1.2); no longer RN3.5 (R4.2)
- net at U7.2 (QC): now also RN4.6 (R3.2); no longer RN3.7 (R2.2)
- net at U7.3 (QD): now also RN4.5 (R4.2); no longer RN3.8 (R1.2)
- net at U7.4 (QE): now also RN3.8 (R1.2); no longer RN4.5 (R4.2)
- net at U7.5 (QF): now also RN3.7 (R2.2); no longer RN4.6 (R3.2)
- net at U7.6 (QG): now also RN3.6 (R3.2); no longer RN4.7 (R2.2)
- net at U7.7 (QH): now also RN3.5 (R4.2); no longer RN4.8 (R1.2)
- net at RN6.1 (R1.1): now also U11.1 (A); no longer U11.6 (LDP)
- net at RN6.2 (R2.1): now also U11.14 (B); no longer U11.13 (G)
- net at RN6.3 (R3.1): now also U11.12 (C); no longer U11.2 (F)
- net at RN6.4 (R4.1): now also U11.10 (D); no longer U11.4 (E)
- net at RN5.1 (R1.1): now also U11.4 (E); no longer U11.10 (D)
- net at RN5.2 (R2.1): now also U11.2 (F); no longer U11.12 (C)
- net at RN5.3 (R3.1): now also U11.13 (G); no longer U11.14 (B)
- net at RN5.4 (R4.1): now also U11.6 (LDP); no longer U11.1 (A)
- net at RN10.1 (R1.1): now also U16.1 (A); no longer U16.4 (H)
- net at RN10.2 (R2.1): now also U16.18 (B); no longer U16.8 (G)
- net at RN10.3 (R3.1): now also U16.16 (C); no longer U16.9 (F)
- net at RN10.4 (R4.1): now also U16.13 (D); no longer U16.10 (E)
Other:
- moved on the sheet: RN1, RN10, RN11, RN12, RN2, RN3, RN4, RN5, RN6, RN7, RN8, RN9
