File: pcb/ws2812.kicad_sch (KiCad schematic)
At the start: 37 parts

Commit message: Laid out and routed PCB
Parts:
- R9: footprint (none) -> Resistor_SMD:R_0402_1005Metric
- renumbered D23 to D16, D22 to D17, D21 to D18, D20 to D19, D19 to D20, D18 to D21, D17 to D22, D16 to D23
Changed lines of the file:
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@@
   (symbol (lib_id "LED:WS2812B") (at 127 86.36 0) (mirror y) (unit 1)
     (in_bom yes) (on_board yes)
-    (property "Reference" "D17" (id 0) (at 121.92 80.01 0))
+    (property "Reference" "D22" (id 0) (at 121.92 80.01 0))
     (property "Value" "WS2812B" (id 1) (at 115.57 84.5693 0)
       (effects (font (size 1.27 1.27)) hide)
@@
   (symbol (lib_id "LED:WS2812B") (at 172.72 86.36 0) (mirror y) (unit 1)
     (in_bom yes) (on_board yes)
-    (property "Reference" "D20" (id 0) (at 167.64 80.01 0))
+    (property "Reference" "D19" (id 0) (at 167.64 80.01 0))
     (property "Value" "WS2812B" (id 1) (at 161.29 84.5693 0)
       (effects (font (size 1.27 1.27)) hide)
@@
   (symbol (lib_id "LED:WS2812B") (at 187.96 86.36 0) (mirror y) (unit 1)
     (in_bom yes) (on_board yes)
-    (property "Reference" "D21" (id 0) (at 182.88 80.01 0))
+    (property "Reference" "D18" (id 0) (at 182.88 80.01 0))
     (property "Value" "WS2812B" (id 1) (at 176.53 84.5693 0)
       (effects (font (size 1.27 1.27)) hide)
@@
   (symbol (lib_id "LED:WS2812B") (at 111.76 86.36 0) (mirror y) (unit 1)
     (in_bom yes) (on_board yes)
-    (property "Reference" "D16" (id 0) (at 106.68 80.01 0))
+    (property "Reference" "D23" (id 0) (at 106.68 80.01 0))
     (property "Value" "WS2812B" (id 1) (at 100.33 84.5693 0)
       (effects (font (size 1.27 1.27)) hide)
@@
   (symbol (lib_id "LED:WS2812B") (at 157.48 86.36 0) (mirror y) (unit 1)
     (in_bom yes) (on_board yes)
-    (property "Reference" "D19" (id 0) (at 152.4 80.01 0))
+    (property "Reference" "D20" (id 0) (at 152.4 80.01 0))
     (property "Value" "WS2812B" (id 1) (at 146.05 84.5693 0)
       (effects (font (size 1.27 1.27)) hide)
@@
   (symbol (lib_id "LED:WS2812B") (at 203.2 86.36 0) (mirror y) (unit 1)
     (in_bom yes) (on_board yes)
-    (property "Reference" "D22" (id 0) (at 198.12 80.01 0))
+    (property "Reference" "D17" (id 0) (at 198.12 80.01 0))
     (property "Value" "WS2812B" (id 1) (at 191.77 84.5693 0)
       (effects (font (size 1.27 1.27)) hide)
@@
     (property "Reference" "R9" (id 0) (at 100.33 59.69 90))
     (property "Value" "330R" (id 1) (at 100.33 62.23 90))
-    (property "Footprint" "" (id 2) (at 100.33 64.77 0)
+    (property "Footprint" "Resistor_SMD:R_0402_1005Metric" (id 2) (at 100.33 64.77 0)
       (effects (font (size 1.27 1.27)) hide)
     )
@@
   (symbol (lib_id "LED:WS2812B") (at 142.24 86.36 0) (mirror y) (unit 1)
     (in_bom yes) (on_board yes)
-    (property "Reference" "D18" (id 0) (at 137.16 80.01 0))
+    (property "Reference" "D21" (id 0) (at 137.16 80.01 0))
     (property "Value" "WS2812B" (id 1) (at 130.81 84.5693 0)
       (effects (font (size 1.27 1.27)) hide)
@@
   (symbol (lib_id "LED:WS2812B") (at 218.44 86.36 0) (mirror y) (unit 1)
     (in_bom yes) (on_board yes)
-    (property "Reference" "D23" (id 0) (at 213.36 80.01 0))
+    (property "Reference" "D16" (id 0) (at 213.36 80.01 0))
     (property "Value" "WS2812B" (id 1) (at 212.09 92.71 0)
       (effects (font (size 1.27 1.27)) hide)
