File: pcb/5v3A_reg.kicad_sch (KiCad schematic)
At the start: 7 parts, among them U2 ADP2303ARDZ-5.0

Commit message: added br24 changes
Changed lines of the file:
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@@
-	)
-	(junction
-		(at 125.73 69.85)
-		(diameter 0)
-		(color 0 0 0 0)
 	)
 	(junction
@@
 	(wire
 		(pts
-			(xy 120.65 69.85) (xy 125.73 69.85)
-		)
-		(stroke
-			(width 0)
-			(type default)
-		)
-	)
-	(wire
-		(pts
 			(xy 161.29 74.93) (xy 163.83 74.93)
 		)
@@
 	(wire
 		(pts
-			(xy 125.73 69.85) (xy 130.81 69.85)
-		)
-		(stroke
-			(width 0)
-			(type default)
-		)
-	)
-	(wire
-		(pts
 			(xy 189.23 74.93) (xy 191.77 74.93)
 		)
@@
 		(pts
 			(xy 181.61 74.93) (xy 182.88 74.93)
+		)
+		(stroke
+			(width 0)
+			(type default)
+		)
+	)
+	(wire
+		(pts
+			(xy 120.65 69.85) (xy 130.81 69.85)
 		)
 		(stroke
@@
 		)
 		(instances
-			(project ""
+			(project "PCB"
 				(path "/68f34db6-b185-48e2-8817-fb07f7d1240e/785c2b5b-0f6e-472e-8e4b-b02b70d5cf35/bb437566-7d32-450d-b77e-65f68738184c"
 					(reference "C102")
@@
 		)
 		(instances
-			(project ""
+			(project "PCB"
 				(path "/68f34db6-b185-48e2-8817-fb07f7d1240e/785c2b5b-0f6e-472e-8e4b-b02b70d5cf35/bb437566-7d32-450d-b77e-65f68738184c"
 					(reference "#PWR0194")
@@
 		)
 		(instances
-			(project ""
+			(project "PCB"
 				(path "/68f34db6-b185-48e2-8817-fb07f7d1240e/785c2b5b-0f6e-472e-8e4b-b02b70d5cf35/bb437566-7d32-450d-b77e-65f68738184c"
 					(reference "#PWR0195")
@@
 		)
 		(instances
-			(project ""
+			(project "PCB"
 				(path "/68f34db6-b185-48e2-8817-fb07f7d1240e/785c2b5b-0f6e-472e-8e4b-b02b70d5cf35/bb437566-7d32-450d-b77e-65f68738184c"
 					(reference "C101")
@@
 		)
 		(instances
-			(project ""
+			(project "PCB"
 				(path "/68f34db6-b185-48e2-8817-fb07f7d1240e/785c2b5b-0f6e-472e-8e4b-b02b70d5cf35/bb437566-7d32-450d-b77e-65f68738184c"
 					(reference "D129")
@@
 			)
 		)
-		(property "Description" "Nonsynchronous Step-Down Regulator 3 Amp Vout 5.0v SOIC-8"
+		(property "Description" ""
 			(at 146.05 74.93 0)
 			(effects
@@
 		)
 		(instances
-			(project ""
+			(project "PCB"
 				(path "/68f34db6-b185-48e2-8817-fb07f7d1240e/785c2b5b-0f6e-472e-8e4b-b02b70d5cf35/bb437566-7d32-450d-b77e-65f68738184c"
 					(reference "U6")
@@
 				(path "/68f34db6-b185-48e2-8817-fb07f7d1240e/785c2b5b-0f6e-472e-8e4b-b02b70d5cf35/f73c095e-19b5-4ca2-82b2-71d1369b65a4"
 					(reference "U2")
-					(unit 1)
-				)
-			)
-		)
-	)
-	(symbol
-		(lib_name "PWR_FLAG_1")
-		(lib_id "power:PWR_FLAG")
-		(at 125.73 69.85 0)
-		(unit 1)
-		(exclude_from_sim no)
-		(in_bom yes)
-		(on_board yes)
-		(dnp no)
-		(fields_autoplaced yes)
-		(property "Reference" "#FLG02"
-			(at 125.73 67.945 0)
-			(effects
-				(font
-					(size 1.27 1.27)
-				)
-				(hide yes)
-			)
-		)
-		(property "Value" "PWR_FLAG"
-			(at 125.73 64.77 0)
-			(effects
-				(font
-					(size 1.27 1.27)
-				)
-			)
-		)
-		(property "Footprint" ""
-			(at 125.73 69.85 0)
-			(effects
-				(font
-					(size 1.27 1.27)
-				)
-				(hide yes)
-			)
-		)
-		(property "Datasheet" "~"
-			(at 125.73 69.85 0)
-			(effects
-				(font
-					(size 1.27 1.27)
-				)
-				(hide yes)
-			)
-		)
-		(property "Description" "Special symbol for telling ERC where power comes from"
-			(at 125.73 69.85 0)
-			(effects
-				(font
-					(size 1.27 1.27)
-				)
-				(hide yes)
-			)
-		)
-		(pin "1"
-		)
-		(instances
-			(project ""
-				(path "/68f34db6-b185-48e2-8817-fb07f7d1240e/785c2b5b-0f6e-472e-8e4b-b02b70d5cf35/bb437566-7d32-450d-b77e-65f68738184c"
-					(reference "#FLG03")
-					(unit 1)
-				)
-				(path "/68f34db6-b185-48e2-8817-fb07f7d1240e/785c2b5b-0f6e-472e-8e4b-b02b70d5cf35/f73c095e-19b5-4ca2-82b2-71d1369b65a4"
-					(reference "#FLG02")
 					(unit 1)
 				)
@@
 		)
 		(instances
-			(project ""
+			(project "PCB"
 				(path "/68f34db6-b185-48e2-8817-fb07f7d1240e/785c2b5b-0f6e-472e-8e4b-b02b70d5cf35/bb437566-7d32-450d-b77e-65f68738184c"
 					(reference "L2")
@@
 		)
 		(instances
-			(project ""
+			(project "PCB"
 				(path "/68f34db6-b185-48e2-8817-fb07f7d1240e/785c2b5b-0f6e-472e-8e4b-b02b70d5cf35/bb437566-7d32-450d-b77e-65f68738184c"
 					(reference "#PWR0192")
@@
 		)
 		(instances
-			(project ""
+			(project "PCB"
 				(path "/68f34db6-b185-48e2-8817-fb07f7d1240e/785c2b5b-0f6e-472e-8e4b-b02b70d5cf35/bb437566-7d32-450d-b77e-65f68738184c"
 					(reference "C100")
@@
 		)
 		(instances
-			(project ""
+			(project "PCB"
 				(path "/68f34db6-b185-48e2-8817-fb07f7d1240e/785c2b5b-0f6e-472e-8e4b-b02b70d5cf35/bb437566-7d32-450d-b77e-65f68738184c"
 					(reference "#PWR0193")
@@
 		)
 		(instances
-			(project ""
+			(project "PCB"
 				(path "/68f34db6-b185-48e2-8817-fb07f7d1240e/785c2b5b-0f6e-472e-8e4b-b02b70d5cf35/bb437566-7d32-450d-b77e-65f68738184c"
 					(reference "#FLG0106")
@@
 		)
 		(instances
-			(project ""
+			(project "PCB"
 				(path "/68f34db6-b185-48e2-8817-fb07f7d1240e/785c2b5b-0f6e-472e-8e4b-b02b70d5cf35/bb437566-7d32-450d-b77e-65f68738184c"
 					(reference "R2")

Commit message: Parts
Parts:
- renumbered C97 to C100, C98 to C101, C99 to C102, D128 to D129, L1 to L2, R1 to R2, U2 to U6
Changed lines of the file:
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@@
 		(on_board yes)
 		(dnp no)
-		(property "Reference" "C99"
+		(property "Reference" "C102"
 			(at 184.15 77.47 0)
 			(effects
@@
 		(dnp no)
 		(fields_autoplaced yes)
-		(property "Reference" "#PWR0190"
+		(property "Reference" "#PWR0194"
 			(at 181.61 88.9 0)
 			(effects
@@
 		(dnp no)
 		(fields_autoplaced yes)
-		(property "Reference" "#PWR0191"
+		(property "Reference" "#PWR0195"
 			(at 163.83 88.9 0)
 			(effects
@@
 		(on_board yes)
 		(dnp no)
-		(property "Reference" "C98"
+		(property "Reference" "C101"
 			(at 163.6268 71.2216 0)
 			(effects
@@
 		(dnp no)
 		(fields_autoplaced yes)
-		(property "Reference" "D128"
+		(property "Reference" "D129"
 			(at 166.37 77.1524 90)
 			(effects
@@
 		(dnp no)
 		(fields_autoplaced yes)
-		(property "Reference" "U2"
+		(property "Reference" "U6"
 			(at 146.05 63.5 0)
 			(effects
@@
 		(dnp no)
 		(fields_autoplaced yes)
-		(property "Reference" "L1"
+		(property "Reference" "L2"
 			(at 173.99 69.85 90)
 			(effects
@@
 		(dnp no)
 		(fields_autoplaced yes)
-		(property "Reference" "#PWR0188"
+		(property "Reference" "#PWR0192"
 			(at 148.59 93.98 0)
 			(effects
@@
 		(on_board yes)
 		(dnp no)
-		(property "Reference" "C97"
+		(property "Reference" "C100"
 			(at 115.57 72.39 0)
 			(effects
@@
 		(dnp no)
 		(fields_autoplaced yes)
-		(property "Reference" "#PWR0189"
+		(property "Reference" "#PWR0193"
 			(at 120.65 81.28 0)
 			(effects
@@
 		(on_board yes)
 		(dnp no)
-		(property "Reference" "#FLG0104"
+		(property "Reference" "#FLG0106"
 			(at 182.88 73.025 0)
 			(effects
@@
 		(on_board yes)
 		(dnp no)
-		(property "Reference" "R1"
+		(property "Reference" "R2"
 			(at 125.73 74.93 0)
 			(effects
