File: pcb/io.kicad_sch (KiCad schematic)
At the start: 46 parts, among them J2 JST B24B-PADSS-F, J4 JST B04B-XASK, U17 ESD224DQA, U18 ESD224DQA, U19 ESD224DQA, U20 ESD224DQA

Commit message: Parts
Parts:
- J2: LCSC (none) -> C5329907
- J4: LCSC (none) -> C160300
- U17, U18, U19, U20: LCSC (none) -> C1981316
Changed lines of the file:
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@@
 			)
 		)
+		(property "LCSC" "C5329907"
+			(at 233.68 62.23 0)
+			(effects
+				(font
+					(size 1.27 1.27)
+				)
+				(hide yes)
+			)
+		)
 		(pin "1"
 		)
@@
 			)
 		)
+		(property "LCSC" "C160300"
+			(at 233.68 91.44 0)
+			(effects
+				(font
+					(size 1.27 1.27)
+				)
+				(hide yes)
+			)
+		)
 		(pin "1"
 		)
@@
 			)
 		)
+		(property "LCSC" "C1981316"
+			(at 96.52 100.33 0)
+			(effects
+				(font
+					(size 1.27 1.27)
+				)
+				(hide yes)
+			)
+		)
 		(pin "1"
 		)
@@
 			)
 		)
+		(property "LCSC" "C1981316"
+			(at 96.52 69.85 0)
+			(effects
+				(font
+					(size 1.27 1.27)
+				)
+				(hide yes)
+			)
+		)
 		(pin "1"
 		)
@@
 			)
 		)
+		(property "LCSC" "C1981316"
+			(at 96.52 163.83 0)
+			(effects
+				(font
+					(size 1.27 1.27)
+				)
+				(hide yes)
+			)
+		)
 		(pin "1"
 		)
@@
 			(at 96.52 132.08 0)
 			(effects
+				(font
+					(size 1.27 1.27)
+				)
+				(hide yes)
+			)
+		)
+		(property "LCSC" "C1981316"
+			(at 96.52 132.08 0)
+			(effects
