File: pcb/led_digit.kicad_sch (KiCad schematic)
At the start: 23 parts

Commit message: added br24 changes
Parts:
- D53, D54, D55, D56, D57, D58, D59, D60, D61, D62, D63, D64, D65, D66, D67: footprint XL-3528RGBW-WS2812B:XL-3528RGBW-WS2812B -> LED_SMD:LED_WS2812B_PLCC4_5.0x5.0mm_P3.2mm
Connections:
- net DATA_IN: now also D67.2 (DOUT); no longer D57.4 (DIN)
- net DATA_OUT: now also D57.4 (DIN); no longer D67.2 (DOUT)
Other:
- note added: "NOTE: DATA_IN goes to DOUT and DATA_OUT goes to DIN This is because the 3529 WS2812 footprint swaps these pins for some god-forsaken reason. And I was way too lazy to redo this whole sub-schematic and make a new symbol just to fix that."

Commit message: Parts
Parts:
- D113: renamed from D53; LCSC (none) -> C22371521
- D114: renamed from D54; LCSC (none) -> C22371521
- D115: renamed from D55; LCSC (none) -> C22371521
- D116: renamed from D56; LCSC (none) -> C22371521
- D117: renamed from D57; LCSC (none) -> C22371521
- D118: renamed from D58; LCSC (none) -> C22371521
- D119: renamed from D59; LCSC (none) -> C22371521
- D120: renamed from D60; LCSC (none) -> C22371521
- D121: renamed from D61; LCSC (none) -> C22371521
- D122: renamed from D62; LCSC (none) -> C22371521
- D123: renamed from D63; LCSC (none) -> C22371521
- D124: renamed from D64; LCSC (none) -> C22371521
- D125: renamed from D65; LCSC (none) -> C22371521
- D126: renamed from D66; LCSC (none) -> C22371521
- D127: renamed from D67; LCSC (none) -> C22371521
- renumbered C57 to C89, C58 to C90, C59 to C91, C60 to C92, C61 to C93, C62 to C94, C63 to C95, C64 to C96
Changed lines of the file:
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@@
 		(dnp no)
 		(fields_autoplaced yes)
-		(property "Reference" "#PWR0143"
+		(property "Reference" "#PWR0183"
 			(at 128.27 127 0)
 			(effects
@@
 		(on_board yes)
 		(dnp no)
-		(property "Reference" "D67"
+		(property "Reference" "D127"
 			(at 161.29 142.24 0)
 			(effects
@@
 			)
 		)
+		(property "LCSC" "C22371521"
+			(at 156.21 148.59 0)
+			(effects
+				(font
+					(size 1.27 1.27)
+				)
+				(hide yes)
+			)
+		)
 		(pin "1"
 		)
@@
 		(on_board yes)
 		(dnp no)
-		(property "Reference" "C61"
+		(property "Reference" "C93"
 			(at 105.2068 166.4716 0)
 			(effects
@@
 		(on_board yes)
 		(dnp no)
-		(property "Reference" "D62"
+		(property "Reference" "D122"
 			(at 125.73 85.09 0)
 			(effects
@@
 			)
 		)
+		(property "LCSC" "C22371521"
+			(at 120.65 91.44 0)
+			(effects
+				(font
+					(size 1.27 1.27)
+				)
+				(hide yes)
+			)
+		)
 		(pin "1"
 		)
@@
 		(on_board yes)
 		(dnp no)
-		(property "Reference" "D57"
+		(property "Reference" "D117"
 			(at 109.22 40.64 0)
 			(effects
@@
 		)
 		(property "Description" ""
+			(at 104.14 46.99 0)
+			(effects
+				(font
+					(size 1.27 1.27)
+				)
+				(hide yes)
+			)
+		)
+		(property "LCSC" "C22371521"
 			(at 104.14 46.99 0)
 			(effects
@@
 		(dnp no)
 		(fields_autoplaced yes)
-		(property "Reference" "#PWR0145"
+		(property "Reference" "#PWR0185"
 			(at 119.38 62.23 0)
 			(effects
@@
 		(on_board yes)
 		(dnp no)
-		(property "Reference" "D66"
+		(property "Reference" "D126"
 			(at 142.24 124.46 90)
 			(effects
@@
 		)
 		(property "Description" ""
+			(at 135.89 119.38 0)
+			(effects
+				(font
+					(size 1.27 1.27)
+				)
+				(hide yes)
+			)
+		)
+		(property "LCSC" "C22371521"
 			(at 135.89 119.38 0)
 			(effects
@@
 		(dnp no)
 		(fields_autoplaced yes)
-		(property "Reference" "#PWR0144"
+		(property "Reference" "#PWR0184"
 			(at 128.27 86.36 0)
 			(effects
@@
 		(dnp no)
 		(fields_autoplaced yes)
-		(property "Reference" "#PWR0146"
+		(property "Reference" "#PWR0186"
 			(at 119.38 153.67 0)
 			(effects
@@
 		(on_board yes)
 		(dnp no)
-		(property "Reference" "D55"
+		(property "Reference" "D115"
 			(at 83.82 57.15 90)
 			(effects
@@
 			)
 		)
+		(property "LCSC" "C22371521"
+			(at 87.63 104.14 0)
+			(effects
+				(font
+					(size 1.27 1.27)
+				)
+				(hide yes)
+			)
+		)
 		(pin "1"
 		)
@@
 		(on_board yes)
 		(dnp no)
-		(property "Reference" "D59"
+		(property "Reference" "D119"
 			(at 110.49 85.09 0)
 			(effects
@@
 			)
 		)
+		(property "LCSC" "C22371521"
+			(at 105.41 91.44 0)
+			(effects
+				(font
+					(size 1.27 1.27)
+				)
+				(hide yes)
+			)
+		)
 		(pin "1"
 		)
@@
 		(on_board yes)
 		(dnp no)
-		(property "Reference" "D53"
+		(property "Reference" "D113"
 			(at 83.82 97.79 90)
 			(effects
@@
 		)
 		(property "Description" ""
+			(at 87.63 63.5 0)
+			(effects
+				(font
+					(size 1.27 1.27)
+				)
+				(hide yes)
+			)
+		)
+		(property "LCSC" "C22371521"
 			(at 87.63 63.5 0)
 			(effects
@@
 		(dnp no)
 		(fields_autoplaced yes)
-		(property "Reference" "#PWR0142"
+		(property "Reference" "#PWR0182"
 			(at 95.25 127 0)
 			(effects
@@
 		(on_board yes)
 		(dnp no)
-		(property "Reference" "C63"
+		(property "Reference" "C95"
 			(at 117.9068 166.4716 0)
 			(effects
@@
 		(on_board yes)
 		(dnp no)
-		(property "Reference" "D54"
+		(property "Reference" "D114"
 			(at 81.28 73.66 0)
 			(effects
@@
 			)
 		)
+		(property "LCSC" "C22371521"
+			(at 87.63 78.74 0)
+			(effects
+				(font
+					(size 1.27 1.27)
+				)
+				(hide yes)
+			)
+		)
 		(pin "1"
 		)
@@
 		(on_board yes)
 		(dnp no)
-		(property "Reference" "C57"
+		(property "Reference" "C89"
 			(at 77.2668 166.4716 0)
 			(effects
@@
 		(dnp no)
 		(fields_autoplaced yes)
-		(property "Reference" "#PWR0138"
+		(property "Reference" "#PWR0178"
 			(at 74.93 176.53 0)
 			(effects
@@
 		(on_board yes)
 		(dnp no)
-		(property "Reference" "D65"
+		(property "Reference" "D125"
 			(at 142.24 109.22 90)
 			(effects
@@
 			)
 		)
+		(property "LCSC" "C22371521"
+			(at 135.89 104.14 0)
+			(effects
+				(font
+					(size 1.27 1.27)
+				)
+				(hide yes)
+			)
+		)
 		(pin "1"
 		)
@@
 		(on_board yes)
 		(dnp no)
-		(property "Reference" "C58"
+		(property "Reference" "C90"
 			(at 86.1568 166.4716 0)
 			(effects
@@
 		(on_board yes)
 		(dnp no)
-		(property "Reference" "D60"
+		(property "Reference" "D120"
 			(at 124.46 40.64 0)
 			(effects
@@
 			)
 		)
+		(property "LCSC" "C22371521"
+			(at 119.38 46.99 0)
+			(effects
+				(font
+					(size 1.27 1.27)
+				)
+				(hide yes)
+			)
+		)
 		(pin "1"
 		)
@@
 		(on_board yes)
 		(dnp no)
-		(property "Reference" "C60"
+		(property "Reference" "C92"
 			(at 98.8568 166.4716 0)
 			(effects
@@
 		(dnp no)
 		(fields_autoplaced yes)
-		(property "Reference" "#PWR0139"
+		(property "Reference" "#PWR0179"
 			(at 120.65 105.41 0)
 			(effects
@@
 		(on_board yes)
 		(dnp no)
-		(property "Reference" "D56"
+		(property "Reference" "D116"
 			(at 83.82 113.03 90)
 			(effects
@@
 			)
 		)
+		(property "LCSC" "C22371521"
+			(at 87.63 119.38 0)
+			(effects
+				(font
+					(size 1.27 1.27)
+				)
+				(hide yes)
+			)
+		)
 		(pin "1"
 		)
@@
 		(on_board yes)
 		(dnp no)
-		(property "Reference" "D63"
+		(property "Reference" "D123"
 			(at 142.24 68.58 90)
 			(effects
@@
 			)
 		)
+		(property "LCSC" "C22371521"
+			(at 135.89 63.5 0)
+			(effects
+				(font
+					(size 1.27 1.27)
+				)
+				(hide yes)
+			)
+		)
 		(pin "1"
 		)
@@
 		(on_board yes)
 		(dnp no)
-		(property "Reference" "C62"
+		(property "Reference" "C94"
 			(at 111.5568 166.4716 0)
 			(effects
@@
 		(on_board yes)
 		(dnp no)
-		(property "Reference" "D64"
+		(property "Reference" "D124"
 			(at 142.24 83.82 90)
 			(effects
@@
 		)
 		(property "Description" ""
+			(at 135.89 78.74 0)
+			(effects
+				(font
+					(size 1.27 1.27)
+				)
+				(hide yes)
+			)
+		)
+		(property "LCSC" "C22371521"
 			(at 135.89 78.74 0)
 			(effects
@@
 		(on_board yes)
 		(dnp no)
-		(property "Reference" "D61"
+		(property "Reference" "D121"
 			(at 114.3 132.08 0)
 			(effects
@@
 			)
 		)
+		(property "LCSC" "C22371521"
+			(at 119.38 138.43 0)
+			(effects
+				(font
+					(size 1.27 1.27)
+				)
+				(hide yes)
+			)
+		)
 		(pin "1"
 		)
@@
 		(on_board yes)
 		(dnp no)
-		(property "Reference" "C59"
+		(property "Reference" "C91"
 			(at 92.5068 166.4716 0)
 			(effects
@@
 		(on_board yes)
 		(dnp no)
-		(property "Reference" "D58"
+		(property "Reference" "D118"
 			(at 99.06 132.08 0)
 			(effects
@@
 		)
 		(property "Description" ""
+			(at 104.14 138.43 0)
+			(effects
+				(font
+					(size 1.27 1.27)
+				)
+				(hide yes)
+			)
+		)
+		(property "LCSC" "C22371521"
 			(at 104.14 138.43 0)
 			(effects
@@
 		(dnp no)
 		(fields_autoplaced yes)
-		(property "Reference" "#PWR0147"
+		(property "Reference" "#PWR0187"
 			(at 156.21 162.56 0)
 			(effects
@@
 		(dnp no)
 		(fields_autoplaced yes)
-		(property "Reference" "#PWR0140"
+		(property "Reference" "#PWR0180"
 			(at 95.25 86.36 0)
 			(effects
@@
 		(on_board yes)
 		(dnp no)
-		(property "Reference" "C64"
+		(property "Reference" "C96"
 			(at 124.2568 166.4716 0)
 			(effects

Commit message: LED Footprints fixed
Parts:
- D113, D114, D115, D116, D117, D118, D119, D120, D121, D122, D123, D124, D125, D126, D127: footprint LED_SMD:LED_WS2812B_PLCC4_5.0x5.0mm_P3.2mm -> LED_SMD:LED_Kingbright_AAA3528ESGCT
Changed lines of the file:
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@@
 			)
 		)
-		(property "Footprint" "LED_SMD:LED_WS2812B_PLCC4_5.0x5.0mm_P3.2mm"
+		(property "Footprint" "LED_SMD:LED_Kingbright_AAA3528ESGCT"
 			(at 157.48 156.21 0)
 			(effects
@@
 			)
 		)
-		(property "Footprint" "LED_SMD:LED_WS2812B_PLCC4_5.0x5.0mm_P3.2mm"
+		(property "Footprint" "LED_SMD:LED_Kingbright_AAA3528ESGCT"
 			(at 121.92 99.06 0)
 			(effects
@@
 			)
 		)
-		(property "Footprint" "LED_SMD:LED_WS2812B_PLCC4_5.0x5.0mm_P3.2mm"
+		(property "Footprint" "LED_SMD:LED_Kingbright_AAA3528ESGCT"
 			(at 105.41 54.61 0)
 			(effects
@@
 			)
 		)
-		(property "Footprint" "LED_SMD:LED_WS2812B_PLCC4_5.0x5.0mm_P3.2mm"
+		(property "Footprint" "LED_SMD:LED_Kingbright_AAA3528ESGCT"
 			(at 128.27 120.65 0)
 			(effects
@@
 			)
 		)
-		(property "Footprint" "LED_SMD:LED_WS2812B_PLCC4_5.0x5.0mm_P3.2mm"
+		(property "Footprint" "LED_SMD:LED_Kingbright_AAA3528ESGCT"
 			(at 95.25 102.87 0)
 			(effects
@@
 			)
 		)
-		(property "Footprint" "LED_SMD:LED_WS2812B_PLCC4_5.0x5.0mm_P3.2mm"
+		(property "Footprint" "LED_SMD:LED_Kingbright_AAA3528ESGCT"
 			(at 106.68 99.06 0)
 			(effects
@@
 			)
 		)
-		(property "Footprint" "LED_SMD:LED_WS2812B_PLCC4_5.0x5.0mm_P3.2mm"
+		(property "Footprint" "LED_SMD:LED_Kingbright_AAA3528ESGCT"
 			(at 95.25 62.23 0)
 			(effects
@@
 			)
 		)
-		(property "Footprint" "LED_SMD:LED_WS2812B_PLCC4_5.0x5.0mm_P3.2mm"
+		(property "Footprint" "LED_SMD:LED_Kingbright_AAA3528ESGCT"
 			(at 95.25 77.47 0)
 			(effects
@@
 			)
 		)
-		(property "Footprint" "LED_SMD:LED_WS2812B_PLCC4_5.0x5.0mm_P3.2mm"
+		(property "Footprint" "LED_SMD:LED_Kingbright_AAA3528ESGCT"
 			(at 128.27 105.41 0)
 			(effects
@@
 			)
 		)
-		(property "Footprint" "LED_SMD:LED_WS2812B_PLCC4_5.0x5.0mm_P3.2mm"
+		(property "Footprint" "LED_SMD:LED_Kingbright_AAA3528ESGCT"
 			(at 120.65 54.61 0)
 			(effects
@@
 			)
 		)
-		(property "Footprint" "LED_SMD:LED_WS2812B_PLCC4_5.0x5.0mm_P3.2mm"
+		(property "Footprint" "LED_SMD:LED_Kingbright_AAA3528ESGCT"
 			(at 95.25 118.11 0)
 			(effects
@@
 			)
 		)
-		(property "Footprint" "LED_SMD:LED_WS2812B_PLCC4_5.0x5.0mm_P3.2mm"
+		(property "Footprint" "LED_SMD:LED_Kingbright_AAA3528ESGCT"
 			(at 128.27 64.77 0)
 			(effects
@@
 			)
 		)
-		(property "Footprint" "LED_SMD:LED_WS2812B_PLCC4_5.0x5.0mm_P3.2mm"
+		(property "Footprint" "LED_SMD:LED_Kingbright_AAA3528ESGCT"
 			(at 128.27 80.01 0)
 			(effects
@@
 			)
 		)
-		(property "Footprint" "LED_SMD:LED_WS2812B_PLCC4_5.0x5.0mm_P3.2mm"
+		(property "Footprint" "LED_SMD:LED_Kingbright_AAA3528ESGCT"
 			(at 118.11 146.05 0)
 			(effects
@@
 			)
 		)
-		(property "Footprint" "LED_SMD:LED_WS2812B_PLCC4_5.0x5.0mm_P3.2mm"
+		(property "Footprint" "LED_SMD:LED_Kingbright_AAA3528ESGCT"
 			(at 102.87 146.05 0)
 			(effects
