File: pcb/power_supply.kicad_sch (KiCad schematic)
At the start: 10 parts, among them U1 AMS1117-3.3

Commit message: added br24 changes
Other:
- moved on the sheet: C4, C5, D1, D2, D5, D6, F1, R3, R4, U1

Commit message: LED Footprints fixed
Parts:
- D5, D6: LCSC C72043 -> C5875739
- F1: LCSC C122965 -> C122964
Changed lines of the file:
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@@
 			)
 		)
-		(property "LCSC" "C122965"
+		(property "LCSC" "C122964"
 			(at 81.28 72.39 0)
 			(effects
@@
 			)
 		)
-		(property "LCSC" "C72043"
+		(property "LCSC" "C5875739"
 			(at 250.19 81.28 0)
 			(effects
@@
 			)
 		)
-		(property "LCSC" "C72043"
+		(property "LCSC" "C5875739"
 			(at 260.35 81.28 0)
 			(effects
